File: PCB_Design/EAGLE/POCKETBEAGLE-POD.sch (EAGLE design)
At the start: 29 parts, among them CN1 1, U1 POCKETBEAGLE, X1 STEREOJACK

Commit message: Documentation Fixes
Other:
- note added: "ENGI301 - LOGAN BALDRIDGE"
- note removed: "ENGI301 - Example"
Changed lines of the file:
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@@
 <sheet>
 <plain>
-<text x="314.96" y="20.32" size="2.54" layer="94">ENGI301 - Example</text>
+<text x="314.96" y="20.32" size="2.54" layer="94">ENGI301 - LOGAN BALDRIDGE</text>
 <text x="332.74" y="5.08" size="2.54" layer="94">1/1</text>
 <wire x1="149.86" y1="12.7" x2="149.86" y2="251.46" width="0.1524" layer="97"/>
